Commit message: Real FR3 deployment on the DROID cell
- Robotiq 2F-85 over the network: socket:// ports, NUC TCP bridge script
- Ready pose with joint 7 = 0; run_hardware moves there on start
- Gripper mount at 0 deg (MJCF + regenerated URDFs) to match the real robot
- Virtual cell walls (floor, front x=0.70, right y=-0.50) in MuJoCo and Viser
- Potential-field repulsion mode for the collision-aware controller
- Configurable FR3 collision reflex thresholds; field capped below them

File: assets/scene/franka_fr3/urdf/fr3_robotiq.urdf (robot description, URDF)
Before this commit: robot fr3, 24 links, 23 joints
Joints:
- joint fr3_gripper_joint: origin xyz=0 0 0 rpy=0 0 -0.785398128 -> xyz=0 0 0 rpy=0 -0 0

File: assets/scene/franka_fr3/urdf/fr3_robotiq_rigid.urdf (robot description, URDF)
Before this commit: robot fr3, 24 links, 23 joints
Joints:
- joint fr3_gripper_joint: origin xyz=0 0 0 rpy=0 0 -0.785398128 -> xyz=0 0 0 rpy=0 -0 0
